Commit message: changed .dae

File: urdf/wheelchair.xacro (robot description, xacro)
@@ -14,44 +14,4 @@
 	<xacro:property name="camera_mass" value="0.1"/>
 	<xacro:property name="hokoyu_mass" value="1e-5"/>
-    <!-- Color of bot -->
-	<gazebo reference="left_wheel_front">
-		<material>Gazebo/Green</material>
-		<kp>1000000.0</kp> <!-- kp and kd for rubber -->
-		<kd>100.0</kd>
-		<mu1>1.0</mu1>
-		<mu2>1.0</mu2>
-		<maxVel>1.0</maxVel>
-		<minDepth>0.00</minDepth>
-	</gazebo>
-	<gazebo reference="left_wheel_back">
-		<material>Gazebo/Green</material>
-		<kp>1000000.0</kp> <!-- kp and kd for rubber -->
-		<kd>100.0</kd>
-		<mu1>1.0</mu1>
-		<mu2>1.0</mu2>
-		<maxVel>1.0</maxVel>
-		<minDepth>0.00</minDepth>
-	</gazebo>
-	<gazebo reference="right_wheel_front">
-		<material>Gazebo/Green</material>
-		<kp>1000000.0</kp> <!-- kp and kd for rubber -->
-		<kd>100.0</kd>
-		<mu1>1.0</mu1>
-		<mu2>1.0</mu2>
-		<maxVel>1.0</maxVel>
-		<minDepth>0.00</minDepth>
-	</gazebo>
-	<gazebo reference="right_wheel_back">
-		<material>Gazebo/Green</material>
-		<kp>1000000.0</kp> <!-- kp and kd for rubber -->
-		<kd>100.0</kd>
-		<mu1>1.0</mu1>
-		<mu2>1.0</mu2>
-		<maxVel>1.0</maxVel>
-		<minDepth>0.00</minDepth>
-	</gazebo>
-	<!--<gazebo reference="right_wheel">
-		<material>Gazebo/Green</material>
-	</gazebo>-->
 	<gazebo reference="camera">
 		<material>Gazebo/Red</material>
@@ -97,12 +57,14 @@
 		</inertial>
 		<visual>
-			<origin xyz="0 0 0" rpy="0 1.5707 1.5707"/>
-			<geometry>
-				<cylinder radius="${robot_wheel_radius}" length="${robot_wheel_length}"/>
-			</geometry>
-		</visual>
-		<collision>
-			<origin xyz="0 0 0" rpy="0 1.5707 1.5707"/>
-			<geometry>
+			<origin xyz="0 0 0" rpy="0 0 0"/>
+			<geometry>
+				<mesh filename="package://wheelchair/meshes/middle_wheel.dae"/>
+				<!--<cylinder radius="${robot_wheel_radius}" length="${robot_wheel_length}"/>-->
+			</geometry>
+		</visual>
+		<collision>
+			<origin xyz="0 0 0" rpy="0 1.5707 1.5707"/>
+			<geometry>
+				<!--<mesh filename="package://wheelchair/meshes/middle_wheel.dae"/>-->
 				<cylinder radius="${robot_wheel_radius}" length="${robot_wheel_length}"/>
 			</geometry>
@@ -121,7 +83,8 @@
 		</inertial>
 		<visual>
-			<origin xyz="0 0 0" rpy="0 1.5707 1.5707"/>
-			<geometry>
-				<cylinder radius="${robot_wheel_radius}" length="${robot_wheel_length}"/>
+			<origin xyz="0 0 0" rpy="0 0 0"/>
+			<geometry>
+				<mesh filename="package://wheelchair/meshes/middle_wheel.dae"/>
+				<!--<cylinder radius="${robot_wheel_radius}" length="${robot_wheel_length}"/>-->
 			</geometry>
 		</visual>
@@ -145,7 +108,8 @@
 		</inertial>
 		<visual>
-			<origin xyz="0 0 0" rpy="0 1.5707 1.5707"/>
-			<geometry>
-				<cylinder radius="${robot_wheel_radius}" length="${robot_wheel_length}"/>
+			<origin xyz="0 0 0" rpy="0 0 0"/>
+			<geometry>
+				<mesh filename="package://wheelchair/meshes/middle_wheel.dae"/>
+				<!--<cylinder radius="${robot_wheel_radius}" length="${robot_wheel_length}"/>-->
 			</geometry>
 		</visual>
@@ -169,7 +133,8 @@
 		</inertial>
 		<visual>
-			<origin xyz="0 0 0" rpy="0 1.5707 1.5707"/>
-			<geometry>
-				<cylinder radius="${robot_wheel_radius}" length="${robot_wheel_length}"/>
+			<origin xyz="0 0 0" rpy="0 0 0"/>
+			<geometry>
+				<mesh filename="package://wheelchair/meshes/middle_wheel.dae"/>
+				<!--<cylinder radius="${robot_wheel_radius}" length="${robot_wheel_length}"/>-->
 			</geometry>
 		</visual>

Commit message: stl

File: urdf/wheelchair.xacro (robot description, xacro)
@@ -59,5 +59,5 @@
 			<origin xyz="0 0 0" rpy="0 0 0"/>
 			<geometry>
-				<mesh filename="package://wheelchair/meshes/middle_wheel.dae"/>
+				<mesh filename="package://wheelchair/meshes/middle_wheel.stl"/>
 				<!--<cylinder radius="${robot_wheel_radius}" length="${robot_wheel_length}"/>-->
 			</geometry>
@@ -85,5 +85,5 @@
 			<origin xyz="0 0 0" rpy="0 0 0"/>
 			<geometry>
-				<mesh filename="package://wheelchair/meshes/middle_wheel.dae"/>
+				<mesh filename="package://wheelchair/meshes/middle_wheel.stl"/>
 				<!--<cylinder radius="${robot_wheel_radius}" length="${robot_wheel_length}"/>-->
 			</geometry>
@@ -110,5 +110,5 @@
 			<origin xyz="0 0 0" rpy="0 0 0"/>
 			<geometry>
-				<mesh filename="package://wheelchair/meshes/middle_wheel.dae"/>
+				<mesh filename="package://wheelchair/meshes/middle_wheel.stl"/>
 				<!--<cylinder radius="${robot_wheel_radius}" length="${robot_wheel_length}"/>-->
 			</geometry>
@@ -135,5 +135,5 @@
 			<origin xyz="0 0 0" rpy="0 0 0"/>
 			<geometry>
-				<mesh filename="package://wheelchair/meshes/middle_wheel.dae"/>
+				<mesh filename="package://wheelchair/meshes/middle_wheel.stl"/>
 				<!--<cylinder radius="${robot_wheel_radius}" length="${robot_wheel_length}"/>-->
 			</geometry>

Commit message: trying my own model

File: urdf/wheelchair.xacro (robot description, xacro)
@@ -14,10 +14,4 @@
 	<xacro:property name="camera_mass" value="0.1"/>
 	<xacro:property name="hokoyu_mass" value="1e-5"/>
-	<gazebo reference="camera">
-		<material>Gazebo/Red</material>
-	</gazebo>
-	<gazebo reference="chassis">
-		<material>Gazebo/Blue</material>
-	</gazebo>
 	<!-- Make Chassis of Bot -->
 	<link name="chassis">
@@ -25,5 +19,5 @@
 		<inertial>
 			<mass value="${robot_chassis_mass}"/>
-      		<origin xyz="0.0 0 0" rpy=" 0 0 0"/>
+      		<origin xyz="1 0 0" rpy=" 0 0 0"/>
       		<inertia
       			ixx="0.147116667" ixy="0" ixz="0"
@@ -33,218 +27,19 @@
 		</inertial>
 		<collision name="collision">
-			<origin xyz="0 0 0.05" rpy=" 0 0 0"/>
+			<origin xyz="1 0 0" rpy=" 0 0 0"/>
 			<geometry>
-				<box size="0.5 0.5 0.2"/>
+				<box size="0.614 0.38 0.165"/>
 			</geometry>
 		</collision>
 		<visual name="chassis_visual">
-			<origin xyz="0 0 0.05" rpy=" 0 0 0"/>
+			<origin xyz="0 0 0" rpy=" 0 0 0"/>
 			<geometry>
-				<box size="0.5 0.5 0.2"/>
+                <mesh filename="package://wheelchair/meshes/full_wheelchair.dae"/>
 			</geometry>
 		</visual>
-	</link>
-	<!-- Right Wheel Back -->
-	<link name="right_wheel_back">
-		<inertial>
-			<mass value="${robot_wheel_mass}"/>
-			<origin xyz="0 0 0" rpy="0 1.5707 1.5707"/>
-			<inertia
-				ixx="0.1" ixy="0.0" ixz="0.0"
-				iyy="0.1" iyz="0.0"
-				izz="0.1"
-			/>
-		</inertial>
-		<visual>
-			<origin xyz="0 0 0" rpy="0 0 0"/>
-			<geometry>
-				<mesh filename="package://wheelchair/meshes/middle_wheel.stl"/>
-				<!--<cylinder radius="${robot_wheel_radius}" length="${robot_wheel_length}"/>-->
-			</geometry>
-		</visual>
-		<collision>
-			<origin xyz="0 0 0" rpy="0 1.5707 1.5707"/>
-			<geometry>
-				<!--<mesh filename="package://wheelchair/meshes/middle_wheel.dae"/>-->
-				<cylinder radius="${robot_wheel_radius}" length="${robot_wheel_length}"/>
-			</geometry>
-		</collision>
-	</link>
-	<!-- Right Wheel Front-->
-	<link name="right_wheel_front">
-		<inertial>
-			<mass value="${robot_wheel_mass}"/>
-			<origin xyz="0 0 0" rpy="0 1.5707 1.5707"/>
-			<inertia
-				ixx="0.1" ixy="0.0" ixz="0.0"
-				iyy="0.1" iyz="0.0"
-				izz="0.1"
-			/>
-		</inertial>
-		<visual>
-			<origin xyz="0 0 0" rpy="0 0 0"/>
-			<geometry>
-				<mesh filename="package://wheelchair/meshes/middle_wheel.stl"/>
-				<!--<cylinder radius="${robot_wheel_radius}" length="${robot_wheel_length}"/>-->
-			</geometry>
-		</visual>
-		<collision>
-			<origin xyz="0 0 0" rpy="0 1.5707 1.5707"/>
-			<geometry>
-				<cylinder radius="${robot_wheel_radius}" length="${robot_wheel_length}"/>
-			</geometry>
-		</collision>
-	</link>
-	<!-- Left wheel Back-->
-	<link name="left_wheel_back">
-		<inertial>
-			<mass value="${robot_wheel_mass}"/>
-			<origin xyz="0 0 0" rpy="0 1.5707 1.5707"/>
-			<inertia
-				ixx="0.1" ixy="0.0" ixz="0.0"
-				iyy="0.1" iyz="0.0"
-				izz="0.1"
-			/>
-		</inertial>
-		<visual>
-			<origin xyz="0 0 0" rpy="0 0 0"/>
-			<geometry>
-				<mesh filename="package://wheelchair/meshes/middle_wheel.stl"/>
-				<!--<cylinder radius="${robot_wheel_radius}" length="${robot_wheel_length}"/>-->
-			</geometry>
-		</visual>
-		<collision>
-			<origin xyz="0 0 0" rpy="0 1.5707 1.5707"/>
-			<geometry>
-				<cylinder radius="${robot_wheel_radius}" length="${robot_wheel_length}"/>
-			</geometry>
-		</collision>
-	</link>
-	<!-- Left wheel Front-->
-	<link name="left_wheel_front">
-		<inertial>
-			<mass value="${robot_wheel_mass}"/>
-			<origin xyz="0 0 0" rpy="0 1.5707 1.5707"/>
-			<inertia
-				ixx="0.1" ixy="0.0" ixz="0.0"
-				iyy="0.1" iyz="0.0"
-				izz="0.1"
-			/>
-		</inertial>
-		<visual>
-			<origin xyz="0 0 0" rpy="0 0 0"/>
-			<geometry>
-				<mesh filename="package://wheelchair/meshes/middle_wheel.stl"/>
-				<!--<cylinder radius="${robot_wheel_radius}" length="${robot_wheel_length}"/>-->
-			</geometry>
-		</visual>
-		<collision>
-			<origin xyz="0 0 0" rpy="0 1.5707 1.5707"/>
-			<geometry>
-				<cylinder radius="${robot_wheel_radius}" length="${robot_wheel_length}"/>
-			</geometry>
-		</collision>
-	</link>
-	<!-- Camera -->
-	<link name="camera">
-		<inertial>
-			<mass value="${camera_mass}"/>
-			<origin xyz="0 0 0" rpy="0 0 0"/>
-			<inertia
-		        ixx="1e-6" ixy="0.0" ixz="0.0"
-		        iyy="1e-6" iyz="0.0"
-		        izz="1e-6"
-		      />
-		</inertial>
-		<visual>
-			<origin xyz="0 0 0" rpy="0 0 0"/>
-			<geometry>
-				<box size="0.05 0.05 0.05"/>
-			</geometry>
-		</visual>
-		<collision>
-			<origin xyz="0 0 0" rpy="0 0 0"/>
-			<geometry>
-				<box size="0.05 0.05 0.05"/>
-			</geometry>
-		</collision>
-	</link>
-	<!-- Hokuyo Lidar -->
-	<link name="hokuyo">
-		<inertial>
-			<mass value="${hokoyu_mass}"/>
-			<origin xyz="0 0 0" rpy="0 0 0"/>
-			<inertia
-		        ixx="1e-6" ixy="0.0" ixz="0.0"
-		        iyy="1e-6" iyz="0.0"
-		        izz="1e-6"
-		      />
-		</inertial>
-		<visual>
-			<origin xyz="0 0 0" rpy="0 0 0"/>
-			<geometry>
-				<box size="0.1 0.1 0.1"/>
-			</geometry>
-		</visual>
-		<collision>
-			<origin xyz="0 0 0" rpy="0 0 0"/>
-			<geometry>
-				<box size="0.1 0.1 0.1"/>
-			</geometry>
-		</collision>
 	</link>
 	<!-- Project center to the ground -->
 	<link name="robot_footprint"></link>
 	<!-- Define Joints -->
-	<!-- Right Wheel Joint Back-->
-	<joint type="continuous" name="right_wheel_hinge_back">
-	    <origin xyz="-0.2 -0.30 0" rpy="0 0 0" />
-	    <parent link="chassis"/>
-	    <child link="right_wheel_back" />
-	    <axis xyz="0 1 0" rpy="0 0 0" />
-	    <limit effort="10000" velocity="1000" />
-	    <dynamics damping="1.0" friction="1.0" />
-	</joint>
-	<!-- Right Wheel Joint Front-->
-	<joint type="continuous" name="right_wheel_hinge_front">
-	    <origin xyz="0.2 -0.30 0" rpy="0 0 0" />
-	    <parent link="chassis"/>
-	    <child link="right_wheel_front" />
-	    <axis xyz="0 1 0" rpy="0 0 0" />
-	    <limit effort="10000" velocity="1000" />
-	    <dynamics damping="1.0" friction="1.0" />
-	</joint>
-	<!-- Left Wheel Joint Back-->
-	<joint type="continuous" name="left_wheel_hinge_back">
-	    <origin xyz="-0.2 0.30 0" rpy="0 0 0" />
-	    <parent link="chassis"/>
-	    <child link="left_wheel_back" />
-	    <axis xyz="0 1 0" rpy="0 0 0" />
-	    <limit effort="10000" velocity="1000" />
-	    <dynamics damping="1.0" friction="1.0" />
-	</joint>
-	<!-- Left Wheel Joint Front-->
-	<joint type="continuous" name="left_wheel_hinge_front">
-	    <origin xyz="0.2 0.30 0" rpy="0 0 0" />
-	    <parent link="chassis"/>
-	    <child link="left_wheel_front" />
-	    <axis xyz="0 1 0" rpy="0 0 0" />
-	    <limit effort="10000" velocity="1000" />
-	    <dynamics damping="1.0" friction="1.0" />
-	</joint>
-	<!-- Camera Joint -->
-	<joint name="camera_joint" type="fixed">
-		<origin xyz="0.26 0 0" rpy="0 0 0" />
-		<parent link="chassis"/>
-		<child link="camera" />
-		<axis xyz="0 1 0"/>
-	</joint>
-	<!-- Hokoyu Joint -->
-	<joint name="hokuyo_joint" type="fixed">
-	    <origin xyz="0.2 0 0.2" rpy="0 0 0" />
-	    <parent link="chassis"/>
-	    <child link="hokuyo" />
-	    <axis xyz="0 1 0"/>
-	</joint>
 	<joint name="robot_footprint_joint" type="fixed">
 		<origin xyz="0 0 0" rpy="0 0 0" />

Commit message: package dependencies

File: urdf/wheelchair.xacro (robot description, xacro)
@@ -19,5 +19,5 @@
 		<inertial>
 			<mass value="${robot_chassis_mass}"/>
-      		<origin xyz="1 0 0" rpy=" 0 0 0"/>
+      		<origin xyz="0.35 0.3 0.2" rpy=" 0 0 0"/>
       		<inertia
       			ixx="0.147116667" ixy="0" ixz="0"
@@ -27,5 +27,5 @@
 		</inertial>
 		<collision name="collision">
-			<origin xyz="1 0 0" rpy=" 0 0 0"/>
+			<origin xyz="0.35 0.3 0.2" rpy=" 0 0 0"/>
 			<geometry>
 				<box size="0.614 0.38 0.165"/>

Commit message: mesh changes

File: urdf/wheelchair.xacro (robot description, xacro)
@@ -4,5 +4,5 @@
 	<xacro:include filename="$(find wheelchair)/urdf/wheelchair.gazebo" />
 	<xacro:property name="robot_name" value="wheelchair" />
-	<xacro:property name="robot_chassis_mass" value="15"/>
+	<xacro:property name="robot_chassis_mass" value="30"/>
 	<xacro:property name="robot_chassis_length" value="0.2"/>
 	<xacro:property name="robot_chassis_radius" value="0.25"/>
@@ -19,5 +19,5 @@
 		<inertial>
 			<mass value="${robot_chassis_mass}"/>
-      		<origin xyz="0.35 0.3 0.2" rpy=" 0 0 0"/>
+      		<origin xyz="0.35 0.29 0.2" rpy=" 0 0 0"/>
       		<inertia
       			ixx="0.147116667" ixy="0" ixz="0"
@@ -27,5 +27,5 @@
 		</inertial>
 		<collision name="collision">
-			<origin xyz="0.35 0.3 0.2" rpy=" 0 0 0"/>
+			<origin xyz="0.35 0.29 0.2" rpy=" 0 0 0"/>
 			<geometry>
 				<box size="0.614 0.38 0.165"/>

Commit message: collada for wheels

File: urdf/wheelchair.xacro (robot description, xacro)
@@ -35,6 +35,30 @@
 			<origin xyz="0 0 0" rpy=" 0 0 0"/>
 			<geometry>
-                <mesh filename="package://wheelchair/meshes/full_wheelchair.dae"/>
+                <mesh filename="package://wheelchair/meshes/wheelchair_chassis.dae"/>
 			</geometry>
+		</visual>
+	</link>
+	<!-- Left Wheel -->
+	<link name="left_wheel">
+		<inertial>
+		<mass value="5"/>
+		<origin xyz="0 0 0" rpy="0 1.5707 1.5707"/>
+		<inertia
+			ixx="0.1" ixy="0.0" ixz="0.0"
+			iyy="0.1" iyz="0.0"
+			izz="0.1"
+		/>
+		</inertial>
+		<collision>
+		<origin xyz="0 0 0" rpy="0 1.5707 1.5707"/>
+		<geometry>
+			<cylinder radius="0.1" length="0.05"/>
+		</geometry>
+		</collision>
+		<visual>
+		<origin xyz="0 0 0" rpy="0 1.5707 1.5707"/>
+		<geometry>
+			<cylinder radius="0.1" length="0.05"/>
+		</geometry>
 		</visual>
 	</link>

Commit message: middle wheels added

File: urdf/wheelchair.xacro (robot description, xacro)
@@ -42,5 +42,5 @@
 	<link name="left_wheel">
 		<inertial>
-		<mass value="5"/>
+		<mass value="3"/>
 		<origin xyz="0 0 0" rpy="0 1.5707 1.5707"/>
 		<inertia
@@ -57,7 +57,31 @@
 		</collision>
 		<visual>
+		<origin xyz="-0.5 -0.5 -0.1" rpy="0 0 0"/>
+		<geometry>
+			<mesh filename="package://wheelchair/meshes/middle_wheel_left.dae"/>
+		</geometry>
+		</visual>
+	</link>
+	<!-- Right Wheel -->
+	<link name="right_wheel">
+		<inertial>
+		<mass value="3"/>
+		<origin xyz="0 0 0" rpy="0 1.5707 1.5707"/>
+		<inertia
+			ixx="0.1" ixy="0.0" ixz="0.0"
+			iyy="0.1" iyz="0.0"
+			izz="0.1"
+		/>
+		</inertial>
+		<collision>
 		<origin xyz="0 0 0" rpy="0 1.5707 1.5707"/>
 		<geometry>
 			<cylinder radius="0.1" length="0.05"/>
+		</geometry>
+		</collision>
+		<visual>
+		<origin xyz="-0.5 0 -0.1" rpy="0 0 0"/>
+		<geometry>
+			<mesh filename="package://wheelchair/meshes/middle_wheel_right.dae"/>
 		</geometry>
 		</visual>
@@ -65,5 +89,5 @@
 	<!-- Project center to the ground -->
 	<link name="robot_footprint"></link>
-	<!-- Define Joints -->
+	<!-- ******** Define Joints ********** -->
 	<joint name="robot_footprint_joint" type="fixed">
 		<origin xyz="0 0 0" rpy="0 0 0" />
@@ -71,3 +95,19 @@
 		<child link="chassis" />
 	</joint>
+	<joint type="continuous" name="left_wheel_hinge">
+		<origin xyz="0.5 0.5 0.1" rpy="0 0 0" />
+		<parent link="chassis"/>
+		<child link="left_wheel" />
+		<axis xyz="0 1 0" rpy="0 0 0" />
+		<limit effort="10000" velocity="1000" />
+		<dynamics damping="1.0" friction="1.0" />
+  	</joint>
+	<joint type="continuous" name="right_wheel_hinge">
+		<origin xyz="0.5 0 0.1" rpy="0 0 0" />
+		<parent link="chassis"/>
+		<child link="right_wheel" />
+		<axis xyz="0 1 0" rpy="0 0 0" />
+		<limit effort="10000" velocity="1000" />
+		<dynamics damping="1.0" friction="1.0" />
+  	</joint>
 </robot>

Commit message: added back wheels

File: urdf/wheelchair.xacro (robot description, xacro)
@@ -81,7 +81,55 @@
 		</collision>
 		<visual>
-		<origin xyz="-0.5 0 -0.1" rpy="0 0 0"/>
+		<origin xyz="-0.5 -0.05 -0.1" rpy="0 0 0"/>
 		<geometry>
 			<mesh filename="package://wheelchair/meshes/middle_wheel_right.dae"/>
+		</geometry>
+		</visual>
+	</link>
+	<!-- Right Wheel Back -->
+	<link name="right_wheel_back">
+		<inertial>
+		<mass value="1"/>
+		<origin xyz="0 0 0" rpy="0 1.5707 1.5707"/>
+		<inertia
+			ixx="0.1" ixy="0.0" ixz="0.0"
+			iyy="0.1" iyz="0.0"
+			izz="0.1"
+		/>
+		</inertial>
+		<collision>
+		<origin xyz="0 0 0" rpy="0 1.5707 1.5707"/>
+		<geometry>
+			<cylinder radius="0.05" length="0.03"/>
+		</geometry>
+		</collision>
+		<visual>
+		<origin xyz="-0.03 -0.05 -0.06" rpy="0 0 0"/>
+		<geometry>
+			<mesh filename="package://wheelchair/meshes/right_wheel_back.dae"/>
+		</geometry>
+		</visual>
+	</link>
+	<!-- Left Wheel Back -->
+	<link name="left_wheel_back">
+		<inertial>
+		<mass value="1"/>
+		<origin xyz="0 0 0" rpy="0 1.5707 1.5707"/>
+		<inertia
+			ixx="0.1" ixy="0.0" ixz="0.0"
+			iyy="0.1" iyz="0.0"
+			izz="0.1"
+		/>
+		</inertial>
+		<collision>
+		<origin xyz="0 0 0" rpy="0 1.5707 1.5707"/>
+		<geometry>
+			<cylinder radius="0.05" length="0.03"/>
+		</geometry>
+		</collision>
+		<visual>
+		<origin xyz="-0.1 -0.5 -0.1" rpy="0 0 0"/>
+		<geometry>
+			<mesh filename="package://wheelchair/meshes/left_wheel_back.dae"/>
 		</geometry>
 		</visual>
@@ -104,5 +152,5 @@
   	</joint>
 	<joint type="continuous" name="right_wheel_hinge">
-		<origin xyz="0.5 0 0.1" rpy="0 0 0" />
+		<origin xyz="0.5 0.05 0.1" rpy="0 0 0" />
 		<parent link="chassis"/>
 		<child link="right_wheel" />
@@ -111,3 +159,19 @@
 		<dynamics damping="1.0" friction="1.0" />
   	</joint>
+	<joint type="continuous" name="right_wheel_hinge_back">
+		<origin xyz="0.03 0.05 0.06" rpy="0 0 0" />
+		<parent link="chassis"/>
+		<child link="right_wheel_back" />
+		<axis xyz="0 1 0" rpy="0 0 0" />
+		<limit effort="10000" velocity="1000" />
+		<dynamics damping="1.0" friction="1.0" />
+  	</joint>
+	  <joint type="continuous" name="left_wheel_hinge_back">
+		<origin xyz="0.1 0.5 0.1" rpy="0 0 0" />
+		<parent link="chassis"/>
+		<child link="left_wheel_back" />
+		<axis xyz="0 1 0" rpy="0 0 0" />
+		<limit effort="10000" velocity="1000" />
+		<dynamics damping="1.0" friction="1.0" />
+  	</joint>
 </robot>

Commit message: fixed wheel collisions and added 4 wheel plugin

File: urdf/wheelchair.xacro (robot description, xacro)
@@ -11,7 +11,5 @@
 	<xacro:property name="robot_wheel_mass" value="5"/>
 	<xacro:property name="robot_wheel_length" value="0.05"/>
-	<xacro:property name="robot_wheel_radius" value="0.1"/>
-	<xacro:property name="camera_mass" value="0.1"/>
-	<xacro:property name="hokoyu_mass" value="1e-5"/>
+	<xacro:property name="middle_wheel_radius" value="0.13"/>
 	<!-- Make Chassis of Bot -->
 	<link name="chassis">
@@ -53,9 +51,9 @@
 		<origin xyz="0 0 0" rpy="0 1.5707 1.5707"/>
 		<geometry>
-			<cylinder radius="0.1" length="0.05"/>
+			<cylinder radius="${middle_wheel_radius}" length="0.05"/>
 		</geometry>
 		</collision>
 		<visual>
-		<origin xyz="-0.5 -0.5 -0.1" rpy="0 0 0"/>
+		<origin xyz="-0.53 -0.525 -0.1275" rpy="0 0 0"/>
 		<geometry>
 			<mesh filename="package://wheelchair/meshes/middle_wheel_left.dae"/>
@@ -77,9 +75,9 @@
 		<origin xyz="0 0 0" rpy="0 1.5707 1.5707"/>
 		<geometry>
-			<cylinder radius="0.1" length="0.05"/>
+			<cylinder radius="${middle_wheel_radius}" length="0.05"/>
 		</geometry>
 		</collision>
 		<visual>
-		<origin xyz="-0.5 -0.05 -0.1" rpy="0 0 0"/>
+		<origin xyz="-0.53 -0.05 -0.1275" rpy="0 0 0"/>
 		<geometry>
 			<mesh filename="package://wheelchair/meshes/middle_wheel_right.dae"/>
@@ -105,5 +103,5 @@
 		</collision>
 		<visual>
-		<origin xyz="-0.03 -0.05 -0.06" rpy="0 0 0"/>
+		<origin xyz="-0.06 -0.055 -0.052" rpy="0 0 0"/>
 		<geometry>
 			<mesh filename="package://wheelchair/meshes/right_wheel_back.dae"/>
@@ -129,5 +127,5 @@
 		</collision>
 		<visual>
-		<origin xyz="-0.1 -0.5 -0.1" rpy="0 0 0"/>
+		<origin xyz="-0.06 -0.525 -0.052" rpy="0 0 0"/>
 		<geometry>
 			<mesh filename="package://wheelchair/meshes/left_wheel_back.dae"/>
@@ -143,6 +141,6 @@
 		<child link="chassis" />
 	</joint>
-	<joint type="continuous" name="left_wheel_hinge">
-		<origin xyz="0.5 0.5 0.1" rpy="0 0 0" />
+	<joint type="continuous" name="left_wheel_hinge_front">
+		<origin xyz="0.53 0.525 0.1275" rpy="0 0 0" />
 		<parent link="chassis"/>
 		<child link="left_wheel" />
@@ -151,6 +149,6 @@
 		<dynamics damping="1.0" friction="1.0" />
   	</joint>
-	<joint type="continuous" name="right_wheel_hinge">
-		<origin xyz="0.5 0.05 0.1" rpy="0 0 0" />
+	<joint type="continuous" name="right_wheel_hinge_front">
+		<origin xyz="0.53 0.05 0.1275" rpy="0 0 0" />
 		<parent link="chassis"/>
 		<child link="right_wheel" />
@@ -160,5 +158,5 @@
   	</joint>
 	<joint type="continuous" name="right_wheel_hinge_back">
-		<origin xyz="0.03 0.05 0.06" rpy="0 0 0" />
+		<origin xyz="0.06 0.055 0.052" rpy="0 0 0" />
 		<parent link="chassis"/>
 		<child link="right_wheel_back" />
@@ -168,5 +166,5 @@
   	</joint>
 	  <joint type="continuous" name="left_wheel_hinge_back">
-		<origin xyz="0.1 0.5 0.1" rpy="0 0 0" />
+		<origin xyz="0.06 0.525 0.052" rpy="0 0 0" />
 		<parent link="chassis"/>
 		<child link="left_wheel_back" />
