Commit message: fixed collisions

File: urdf/wheelchair.xacro (robot description, xacro)
@@ -5,11 +5,7 @@
 	<xacro:property name="robot_name" value="wheelchair" />
 	<xacro:property name="robot_chassis_mass" value="30"/>
-	<xacro:property name="robot_chassis_length" value="0.2"/>
-	<xacro:property name="robot_chassis_radius" value="0.25"/>
-	<xacro:property name="robot_caster_wheel_radius" value="0.05"/>
-	<xacro:property name="robot_caster_wheel_radius_collision" value="0.0499"/>
-	<xacro:property name="robot_wheel_mass" value="5"/>
-	<xacro:property name="robot_wheel_length" value="0.05"/>
+	<xacro:property name="middle_wheel_mass" value="3"/>
 	<xacro:property name="middle_wheel_radius" value="0.13"/>
+	<xacro:property name="rear_wheel_radius" value="0.06"/>
 	<!-- Make Chassis of Bot -->
 	<link name="chassis">
@@ -40,5 +36,5 @@
 	<link name="left_wheel">
 		<inertial>
-		<mass value="3"/>
+		<mass value="${middle_wheel_mass}"/>
 		<origin xyz="0 0 0" rpy="0 1.5707 1.5707"/>
 		<inertia
@@ -55,5 +51,5 @@
 		</collision>
 		<visual>
-		<origin xyz="-0.53 -0.525 -0.1275" rpy="0 0 0"/>
+		<origin xyz="-0.52 -0.525 -0.1275" rpy="0 0 0"/>
 		<geometry>
 			<mesh filename="package://wheelchair/meshes/middle_wheel_left.dae"/>
@@ -64,5 +60,5 @@
 	<link name="right_wheel">
 		<inertial>
-		<mass value="3"/>
+		<mass value="${middle_wheel_mass}"/>
 		<origin xyz="0 0 0" rpy="0 1.5707 1.5707"/>
 		<inertia
@@ -79,5 +75,5 @@
 		</collision>
 		<visual>
-		<origin xyz="-0.53 -0.05 -0.1275" rpy="0 0 0"/>
+		<origin xyz="-0.52 -0.05 -0.1275" rpy="0 0 0"/>
 		<geometry>
 			<mesh filename="package://wheelchair/meshes/middle_wheel_right.dae"/>
@@ -99,9 +95,9 @@
 		<origin xyz="0 0 0" rpy="0 1.5707 1.5707"/>
 		<geometry>
-			<cylinder radius="0.05" length="0.03"/>
+			<cylinder radius="${rear_wheel_radius}" length="0.03"/>
 		</geometry>
 		</collision>
 		<visual>
-		<origin xyz="-0.06 -0.055 -0.052" rpy="0 0 0"/>
+		<origin xyz="-0.06 -0.055 -0.062" rpy="0 0 0"/>
 		<geometry>
 			<mesh filename="package://wheelchair/meshes/right_wheel_back.dae"/>
@@ -123,9 +119,9 @@
 		<origin xyz="0 0 0" rpy="0 1.5707 1.5707"/>
 		<geometry>
-			<cylinder radius="0.05" length="0.03"/>
+			<cylinder radius="${rear_wheel_radius}" length="0.03"/>
 		</geometry>
 		</collision>
 		<visual>
-		<origin xyz="-0.06 -0.525 -0.052" rpy="0 0 0"/>
+		<origin xyz="-0.06 -0.525 -0.062" rpy="0 0 0"/>
 		<geometry>
 			<mesh filename="package://wheelchair/meshes/left_wheel_back.dae"/>
@@ -142,5 +138,5 @@
 	</joint>
 	<joint type="continuous" name="left_wheel_hinge_front">
-		<origin xyz="0.53 0.525 0.1275" rpy="0 0 0" />
+		<origin xyz="0.52 0.525 0.1275" rpy="0 0 0" />
 		<parent link="chassis"/>
 		<child link="left_wheel" />
@@ -150,5 +146,5 @@
   	</joint>
 	<joint type="continuous" name="right_wheel_hinge_front">
-		<origin xyz="0.53 0.05 0.1275" rpy="0 0 0" />
+		<origin xyz="0.52 0.05 0.1275" rpy="0 0 0" />
 		<parent link="chassis"/>
 		<child link="right_wheel" />
@@ -158,5 +154,5 @@
   	</joint>
 	<joint type="continuous" name="right_wheel_hinge_back">
-		<origin xyz="0.06 0.055 0.052" rpy="0 0 0" />
+		<origin xyz="0.06 0.055 0.062" rpy="0 0 0" />
 		<parent link="chassis"/>
 		<child link="right_wheel_back" />
@@ -166,5 +162,5 @@
   	</joint>
 	  <joint type="continuous" name="left_wheel_hinge_back">
-		<origin xyz="0.06 0.525 0.052" rpy="0 0 0" />
+		<origin xyz="0.06 0.525 0.062" rpy="0 0 0" />
 		<parent link="chassis"/>
 		<child link="left_wheel_back" />

Commit message: fixed collision with mesh geometry

File: urdf/wheelchair.xacro (robot description, xacro)
@@ -6,6 +6,7 @@
 	<xacro:property name="robot_chassis_mass" value="30"/>
 	<xacro:property name="middle_wheel_mass" value="3"/>
-	<xacro:property name="middle_wheel_radius" value="0.13"/>
-	<xacro:property name="rear_wheel_radius" value="0.06"/>
+	<xacro:property name="middle_wheel_radius" value="0.128"/>
+	<xacro:property name="rear_wheel_radius" value="0.058"/>
+	<xacro:property name="rear_wheel_length" value="0.025"/>
 	<!-- Make Chassis of Bot -->
 	<link name="chassis">
@@ -51,5 +52,5 @@
 		</collision>
 		<visual>
-		<origin xyz="-0.52 -0.525 -0.1275" rpy="0 0 0"/>
+		<origin xyz="-0.523 -0.525 -0.128" rpy="0 0 0"/>
 		<geometry>
 			<mesh filename="package://wheelchair/meshes/middle_wheel_left.dae"/>
@@ -75,5 +76,5 @@
 		</collision>
 		<visual>
-		<origin xyz="-0.52 -0.05 -0.1275" rpy="0 0 0"/>
+		<origin xyz="-0.523 -0.05 -0.128" rpy="0 0 0"/>
 		<geometry>
 			<mesh filename="package://wheelchair/meshes/middle_wheel_right.dae"/>
@@ -93,11 +94,12 @@
 		</inertial>
 		<collision>
-		<origin xyz="0 0 0" rpy="0 1.5707 1.5707"/>
+		<origin xyz="-0.06 -0.053 -0.062" rpy="0 0 0"/>
 		<geometry>
-			<cylinder radius="${rear_wheel_radius}" length="0.03"/>
+			<mesh filename="package://wheelchair/meshes/right_wheel_back.dae"/>
+			<!--<cylinder radius="${rear_wheel_radius}" length="${rear_wheel_length}"/>-->
 		</geometry>
 		</collision>
 		<visual>
-		<origin xyz="-0.06 -0.055 -0.062" rpy="0 0 0"/>
+		<origin xyz="-0.06 -0.053 -0.062" rpy="0 0 0"/>
 		<geometry>
 			<mesh filename="package://wheelchair/meshes/right_wheel_back.dae"/>
@@ -119,5 +121,5 @@
 		<origin xyz="0 0 0" rpy="0 1.5707 1.5707"/>
 		<geometry>
-			<cylinder radius="${rear_wheel_radius}" length="0.03"/>
+			<cylinder radius="${rear_wheel_radius}" length="${rear_wheel_length}"/>
 		</geometry>
 		</collision>
@@ -138,5 +140,5 @@
 	</joint>
 	<joint type="continuous" name="left_wheel_hinge_front">
-		<origin xyz="0.52 0.525 0.1275" rpy="0 0 0" />
+		<origin xyz="0.523 0.525 0.128" rpy="0 0 0" />
 		<parent link="chassis"/>
 		<child link="left_wheel" />
@@ -146,5 +148,5 @@
   	</joint>
 	<joint type="continuous" name="right_wheel_hinge_front">
-		<origin xyz="0.52 0.05 0.1275" rpy="0 0 0" />
+		<origin xyz="0.523 0.05 0.128" rpy="0 0 0" />
 		<parent link="chassis"/>
 		<child link="right_wheel" />
@@ -154,5 +156,5 @@
   	</joint>
 	<joint type="continuous" name="right_wheel_hinge_back">
-		<origin xyz="0.06 0.055 0.062" rpy="0 0 0" />
+		<origin xyz="0.06 0.053 0.062" rpy="0 0 0" />
 		<parent link="chassis"/>
 		<child link="right_wheel_back" />

Commit message: wheels as cylinders

File: urdf/wheelchair.xacro (robot description, xacro)
@@ -52,5 +52,5 @@
 		</collision>
 		<visual>
-		<origin xyz="-0.523 -0.525 -0.128" rpy="0 0 0"/>
+		<origin xyz="-0.523 -0.525 -0.13" rpy="0 0 0"/>
 		<geometry>
 			<mesh filename="package://wheelchair/meshes/middle_wheel_left.dae"/>
@@ -76,5 +76,5 @@
 		</collision>
 		<visual>
-		<origin xyz="-0.523 -0.05 -0.128" rpy="0 0 0"/>
+		<origin xyz="-0.523 -0.05 -0.13" rpy="0 0 0"/>
 		<geometry>
 			<mesh filename="package://wheelchair/meshes/middle_wheel_right.dae"/>
@@ -94,8 +94,7 @@
 		</inertial>
 		<collision>
-		<origin xyz="-0.06 -0.053 -0.062" rpy="0 0 0"/>
+		<origin xyz="0 0 0" rpy="0 1.5707 1.5707"/>
 		<geometry>
-			<mesh filename="package://wheelchair/meshes/right_wheel_back.dae"/>
-			<!--<cylinder radius="${rear_wheel_radius}" length="${rear_wheel_length}"/>-->
+			<cylinder radius="${rear_wheel_radius}" length="${rear_wheel_length}"/>
 		</geometry>
 		</collision>
@@ -140,5 +139,5 @@
 	</joint>
 	<joint type="continuous" name="left_wheel_hinge_front">
-		<origin xyz="0.523 0.525 0.128" rpy="0 0 0" />
+		<origin xyz="0.523 0.525 0.13" rpy="0 0 0" />
 		<parent link="chassis"/>
 		<child link="left_wheel" />
@@ -148,5 +147,5 @@
   	</joint>
 	<joint type="continuous" name="right_wheel_hinge_front">
-		<origin xyz="0.523 0.05 0.128" rpy="0 0 0" />
+		<origin xyz="0.523 0.05 0.13" rpy="0 0 0" />
 		<parent link="chassis"/>
 		<child link="right_wheel" />

Commit message: major update in URDF

File: urdf/wheelchair.xacro (robot description, xacro)
@@ -4,9 +4,20 @@
 	<xacro:include filename="$(find wheelchair)/urdf/wheelchair.gazebo" />
 	<xacro:property name="robot_name" value="wheelchair" />
-	<xacro:property name="robot_chassis_mass" value="30"/>
-	<xacro:property name="middle_wheel_mass" value="3"/>
+	<xacro:property name="robot_chassis_mass" value="50"/>
+	<xacro:property name="middle_wheel_mass" value="15"/>
 	<xacro:property name="middle_wheel_radius" value="0.128"/>
-	<xacro:property name="rear_wheel_radius" value="0.058"/>
+	<xacro:property name="rear_wheel_radius" value="0.059"/>
 	<xacro:property name="rear_wheel_length" value="0.025"/>
+	<xacro:property name="rear_wheel_mass" value="3"/>
+	<xacro:property name="rear_wheel_support_mass" value="1"/>
+	<!-- Axis Values-->
+	<xacro:property name="z_wheel_support" value="0.125"/>
+	<xacro:property name="z_back_wheel" value="0.059"/>
+	<xacro:property name="z_back_diff" value="-0.066"/> <!-- Equals to: (z_back_wheel - z_wheel_support) -->
+	<xacro:property name="x_wheel_support" value="0.085"/>
+	<xacro:property name="x_back_wheel" value="0.06"/>
+	<xacro:property name="x_back_diff" value="-0.025"/> <!-- Equals to: (x_back_wheel - x_wheel_support) -->
+	<xacro:property name="y_right_wheels_and_support" value="0.051"/>
+	<xacro:property name="y_left_wheels_and_support" value="0.525"/>
 	<!-- Make Chassis of Bot -->
 	<link name="chassis">
@@ -22,7 +33,7 @@
 		</inertial>
 		<collision name="collision">
-			<origin xyz="0.35 0.29 0.2" rpy=" 0 0 0"/>
+			<origin xyz="0 0 0" rpy=" 0 0 0"/>
 			<geometry>
-				<box size="0.614 0.38 0.165"/>
+				<mesh filename="package://wheelchair/meshes/chassis_motor.dae"/>
 			</geometry>
 		</collision>
@@ -30,5 +41,5 @@
 			<origin xyz="0 0 0" rpy=" 0 0 0"/>
 			<geometry>
-                <mesh filename="package://wheelchair/meshes/wheelchair_chassis.dae"/>
+                <mesh filename="package://wheelchair/meshes/chassis_motor.dae"/>
 			</geometry>
 		</visual>
@@ -52,5 +63,5 @@
 		</collision>
 		<visual>
-		<origin xyz="-0.523 -0.525 -0.13" rpy="0 0 0"/>
+		<origin xyz="-0.523 -${y_left_wheels_and_support} -0.13" rpy="0 0 0"/>
 		<geometry>
 			<mesh filename="package://wheelchair/meshes/middle_wheel_left.dae"/>
@@ -76,5 +87,5 @@
 		</collision>
 		<visual>
-		<origin xyz="-0.523 -0.05 -0.13" rpy="0 0 0"/>
+		<origin xyz="-0.523 -${y_right_wheels_and_support} -0.13" rpy="0 0 0"/>
 		<geometry>
 			<mesh filename="package://wheelchair/meshes/middle_wheel_right.dae"/>
@@ -85,5 +96,5 @@
 	<link name="right_wheel_back">
 		<inertial>
-		<mass value="1"/>
+		<mass value="${rear_wheel_mass}"/>
 		<origin xyz="0 0 0" rpy="0 1.5707 1.5707"/>
 		<inertia
@@ -100,5 +111,5 @@
 		</collision>
 		<visual>
-		<origin xyz="-0.06 -0.053 -0.062" rpy="0 0 0"/>
+		<origin xyz="-${x_back_wheel} -${y_right_wheels_and_support} -${z_back_wheel}" rpy="0 0 0"/>
 		<geometry>
 			<mesh filename="package://wheelchair/meshes/right_wheel_back.dae"/>
@@ -109,5 +120,5 @@
 	<link name="left_wheel_back">
 		<inertial>
-		<mass value="1"/>
+		<mass value="${rear_wheel_mass}"/>
 		<origin xyz="0 0 0" rpy="0 1.5707 1.5707"/>
 		<inertia
@@ -124,7 +135,55 @@
 		</collision>
 		<visual>
-		<origin xyz="-0.06 -0.525 -0.062" rpy="0 0 0"/>
+		<origin xyz="-${x_back_wheel} -${y_left_wheels_and_support} -${z_back_wheel}" rpy="0 0 0"/>
 		<geometry>
 			<mesh filename="package://wheelchair/meshes/left_wheel_back.dae"/>
+		</geometry>
+		</visual>
+	</link>
+	<!-- Left Wheel Support -->
+	<link name="left_wheel_support">
+		<inertial>
+		<mass value="${rear_wheel_support_mass}"/>
+		<origin xyz="0 0 0" rpy="0 1.5707 1.5707"/>
+		<inertia
+			ixx="0.1" ixy="0.0" ixz="0.0"
+			iyy="0.1" iyz="0.0"
+			izz="0.1"
+		/>
+		</inertial>
+		<collision>
+		<origin xyz="-${x_wheel_support} -${y_left_wheels_and_support} -${z_wheel_support}" rpy="0 0 0"/>
+		<geometry>
+			<mesh filename="package://wheelchair/meshes/left_wheel_support.dae"/>
+		</geometry>
+		</collision>
+		<visual>
+		<origin xyz="-${x_wheel_support} -${y_left_wheels_and_support} -${z_wheel_support}" rpy="0 0 0"/>
+		<geometry>
+			<mesh filename="package://wheelchair/meshes/left_wheel_support.dae"/>
+		</geometry>
+		</visual>
+	</link>
+	<!-- Right Wheel Support -->
+	<link name="right_wheel_support">
+		<inertial>
+		<mass value="${rear_wheel_support_mass}"/>
+		<origin xyz="0 0 0" rpy="0 1.5707 1.5707"/>
+		<inertia
+			ixx="0.1" ixy="0.0" ixz="0.0"
+			iyy="0.1" iyz="0.0"
+			izz="0.1"
+		/>
+		</inertial>
+		<collision>
+		<origin xyz="-${x_wheel_support} -${y_right_wheels_and_support} -${z_wheel_support}" rpy="0 0 0"/>
+		<geometry>
+			<mesh filename="package://wheelchair/meshes/right_wheel_support.dae"/>
+		</geometry>
+		</collision>
+		<visual>
+		<origin xyz="-${x_wheel_support} -${y_right_wheels_and_support} -${z_wheel_support}" rpy="0 0 0"/>
+		<geometry>
+			<mesh filename="package://wheelchair/meshes/right_wheel_support.dae"/>
 		</geometry>
 		</visual>
@@ -138,6 +197,6 @@
 		<child link="chassis" />
 	</joint>
-	<joint type="continuous" name="left_wheel_hinge_front">
-		<origin xyz="0.523 0.525 0.13" rpy="0 0 0" />
+	<joint type="continuous" name="left_wheel_front_joint">
+		<origin xyz="0.523 ${y_left_wheels_and_support} 0.13" rpy="0 0 0" />
 		<parent link="chassis"/>
 		<child link="left_wheel" />
@@ -146,6 +205,6 @@
 		<dynamics damping="1.0" friction="1.0" />
   	</joint>
-	<joint type="continuous" name="right_wheel_hinge_front">
-		<origin xyz="0.523 0.05 0.13" rpy="0 0 0" />
+	<joint type="continuous" name="right_wheel_front_joint">
+		<origin xyz="0.523 ${y_right_wheels_and_support} 0.13" rpy="0 0 0" />
 		<parent link="chassis"/>
 		<child link="right_wheel" />
@@ -154,7 +213,31 @@
 		<dynamics damping="1.0" friction="1.0" />
   	</joint>
-	<joint type="continuous" name="right_wheel_hinge_back">
-		<origin xyz="0.06 0.053 0.062" rpy="0 0 0" />
-		<parent link="chassis"/>
+	<joint type="continuous" name="right_wheel_support_joint">
+		<origin xyz="${x_wheel_support} ${y_right_wheels_and_support} ${z_wheel_support}" rpy="0 0 0" />
+		<parent link="chassis"/>
+		<child link="right_wheel_support" />
+		<axis xyz="0 0 1" rpy="0 0 0" />
+		<limit effort="10000" velocity="1000" />
+		<dynamics damping="1.0" friction="1.0" />
+  	</joint>
+	<joint type="continuous" name="left_wheel_support_joint">
+		<origin xyz="${x_wheel_support} ${y_left_wheels_and_support} ${z_wheel_support}" rpy="0 0 0" />
+		<parent link="chassis"/>
+		<child link="left_wheel_support" />
+		<axis xyz="0 0 1" rpy="0 0 0" />
+		<limit effort="10000" velocity="1000" />
+		<dynamics damping="1.0" friction="1.0" />
+  	</joint>
+	<joint type="continuous" name="rear_left_wheel_joint">
+		<origin xyz="${x_back_diff} 0 ${z_back_diff}" rpy="0 0 0" />
+		<parent link="left_wheel_support"/>
+		<child link="left_wheel_back" />
+		<axis xyz="0 1 0" rpy="0 0 0" />
+		<limit effort="10000" velocity="1000" />
+		<dynamics damping="1.0" friction="1.0" />
+  	</joint>
+	<joint type="continuous" name="rear_right_wheel_joint">
+		<origin xyz="${x_back_diff} 0 ${z_back_diff}" rpy="0 0 0" />
+		<parent link="right_wheel_support"/>
 		<child link="right_wheel_back" />
 		<axis xyz="0 1 0" rpy="0 0 0" />
@@ -162,11 +245,3 @@
 		<dynamics damping="1.0" friction="1.0" />
   	</joint>
-	  <joint type="continuous" name="left_wheel_hinge_back">
-		<origin xyz="0.06 0.525 0.062" rpy="0 0 0" />
-		<parent link="chassis"/>
-		<child link="left_wheel_back" />
-		<axis xyz="0 1 0" rpy="0 0 0" />
-		<limit effort="10000" velocity="1000" />
-		<dynamics damping="1.0" friction="1.0" />
-  	</joint>
 </robot>

Commit message: Added controlers and fixed wheels

File: urdf/wheelchair.xacro (robot description, xacro)
@@ -2,22 +2,22 @@
 <robot name="wheelchair" xmlns:xacro="http://www.ros.org/wiki/xacro">
     <!-- Motor, Camera and Lidar Simulation -->
-	<xacro:include filename="$(find wheelchair)/urdf/wheelchair.gazebo" />
+	<!--<xacro:include filename="$(find wheelchair)/urdf/wheelchair.gazebo" />-->
 	<xacro:property name="robot_name" value="wheelchair" />
 	<xacro:property name="robot_chassis_mass" value="50"/>
 	<xacro:property name="middle_wheel_mass" value="15"/>
 	<xacro:property name="middle_wheel_radius" value="0.128"/>
-	<xacro:property name="rear_wheel_radius" value="0.059"/>
+	<xacro:property name="rear_wheel_radius" value="0.060"/>
 	<xacro:property name="rear_wheel_length" value="0.025"/>
 	<xacro:property name="rear_wheel_mass" value="3"/>
-	<xacro:property name="rear_wheel_support_mass" value="1"/>
+	<xacro:property name="rear_wheel_support_mass" value="2"/>
 	<!-- Axis Values-->
 	<xacro:property name="z_wheel_support" value="0.125"/>
-	<xacro:property name="z_back_wheel" value="0.059"/>
-	<xacro:property name="z_back_diff" value="-0.066"/> <!-- Equals to: (z_back_wheel - z_wheel_support) -->
-	<xacro:property name="x_wheel_support" value="0.085"/>
+	<xacro:property name="z_back_wheel" value="0.062"/>
+	<xacro:property name="z_back_diff" value="-0.063"/> <!-- Equals to: (z_back_wheel - z_wheel_support) -->
+	<xacro:property name="x_wheel_support" value="0.083"/>
 	<xacro:property name="x_back_wheel" value="0.06"/>
-	<xacro:property name="x_back_diff" value="-0.025"/> <!-- Equals to: (x_back_wheel - x_wheel_support) -->
+	<xacro:property name="x_back_diff" value="-0.023"/> <!-- Equals to: (x_back_wheel - x_wheel_support) -->
 	<xacro:property name="y_right_wheels_and_support" value="0.051"/>
-	<xacro:property name="y_left_wheels_and_support" value="0.525"/>
+	<xacro:property name="y_left_wheels_and_support" value="0.527"/>
 	<!-- Make Chassis of Bot -->
 	<link name="chassis">
@@ -245,3 +245,29 @@
 		<dynamics damping="1.0" friction="1.0" />
   	</joint>
+	<transmission name="left_wheel_trans">
+		<type>transmission_interface/SimpleTransmission</type>
+		<actuator name="left_wheel_motor">
+			<hardwareInterface>EffortJointInterface</hardwareInterface>
+			<mechanicalReduction>1</mechanicalReduction>
+		</actuator>
+		<joint name="left_wheel_front_joint">
+		<hardwareInterface>VelocityJointInterface</hardwareInterface>
+		</joint>
+ 	</transmission>
+	<transmission name="right_wheel_trans">
+		<type>transmission_interface/SimpleTransmission</type>
+		<actuator name="right_wheel_motor">
+			<hardwareInterface>EffortJointInterface</hardwareInterface>
+			<mechanicalReduction>1</mechanicalReduction>
+		</actuator>
+		<joint name="right_wheel_front_joint">
+		<hardwareInterface>VelocityJointInterface</hardwareInterface>
+		</joint>
+ 	</transmission>
+	 <!-- Add ROS plugin so we can interact with our robot -->
+	<gazebo>
+		<plugin name="gazebo_ros_control" filename="libgazebo_ros_control.so">
+		<robotNamespace>/</robotNamespace>
+		</plugin>
+	</gazebo>
 </robot>
