Commit message: added upper chassis

File: urdf/wheelchair.xacro (robot description, xacro)
@@ -4,5 +4,6 @@
 	<!--<xacro:include filename="$(find wheelchair)/urdf/wheelchair.gazebo" />-->
 	<xacro:property name="robot_name" value="wheelchair" />
-	<xacro:property name="robot_chassis_mass" value="50"/>
+	<xacro:property name="chassis_mass" value="50"/>
+	<xacro:property name="upper_chassis_mass" value="30"/>
 	<xacro:property name="middle_wheel_mass" value="15"/>
 	<xacro:property name="middle_wheel_radius" value="0.128"/>
@@ -20,9 +21,12 @@
 	<xacro:property name="y_right_wheels_and_support" value="0.051"/>
 	<xacro:property name="y_left_wheels_and_support" value="0.527"/>
+	<xacro:property name="x_upper_chassis" value="0.42"/>
+	<xacro:property name="y_upper_chassis" value="0.29"/>
+	<xacro:property name="z_upper_chassis" value="0.4"/>
 	<!-- Make Chassis of Bot -->
 	<link name="chassis">
 		<pose>0 0 0.1 0 0 0</pose>
 		<inertial>
-			<mass value="${robot_chassis_mass}"/>
+			<mass value="${chassis_mass}"/>
       		<origin xyz="0.35 0.29 0.2" rpy=" 0 0 0"/>
       		<inertia
@@ -45,26 +49,49 @@
 		</visual>
 	</link>
+	<link name="upper_chassis">
+		<inertial>
+			<mass value="${upper_chassis_mass}"/>
+      		<origin xyz="0 0 0" rpy=" 0 0 0"/>
+      		<inertia
+      			ixx="0.147116667" ixy="0" ixz="0"
+      			iyy="0.334951167" iyz="0"
+      			izz="0.3978345"
+      		/>
+		</inertial>
+		<collision>
+			<origin xyz="-${x_upper_chassis} -${y_upper_chassis} -${y_upper_chassis}" rpy="0 0 0"/>
+			<geometry>
+				<mesh filename="package://wheelchair/meshes/upper_chassis.dae"/>
+			</geometry>
+		</collision>
+		<visual>
+			<origin xyz="-${x_upper_chassis} -${y_upper_chassis} -${y_upper_chassis}" rpy="0 0 0"/>
+			<geometry>
+				<mesh filename="package://wheelchair/meshes/upper_chassis.dae"/>
+			</geometry>
+		</visual>
+	</link>
 	<!-- Left Wheel -->
 	<link name="left_wheel">
 		<inertial>
-		<mass value="${middle_wheel_mass}"/>
-		<origin xyz="0 0 0" rpy="0 1.5707 1.5707"/>
-		<inertia
-			ixx="0.1" ixy="0.0" ixz="0.0"
-			iyy="0.1" iyz="0.0"
-			izz="0.1"
-		/>
-		</inertial>
-		<collision>
-		<origin xyz="0 0 0" rpy="0 1.5707 1.5707"/>
-		<geometry>
-			<cylinder radius="${middle_wheel_radius}" length="0.05"/>
-		</geometry>
-		</collision>
-		<visual>
-		<origin xyz="-0.523 -${y_left_wheels_and_support} -0.13" rpy="0 0 0"/>
-		<geometry>
-			<mesh filename="package://wheelchair/meshes/middle_wheel_left.dae"/>
-		</geometry>
+			<mass value="${middle_wheel_mass}"/>
+			<origin xyz="0 0 0" rpy="0 1.5707 1.5707"/>
+			<inertia
+				ixx="0.1" ixy="0.0" ixz="0.0"
+				iyy="0.1" iyz="0.0"
+				izz="0.1"
+			/>
+		</inertial>
+		<collision>
+			<origin xyz="0 0 0" rpy="0 1.5707 1.5707"/>
+			<geometry>
+				<cylinder radius="${middle_wheel_radius}" length="0.05"/>
+			</geometry>
+		</collision>
+		<visual>
+			<origin xyz="-0.523 -${y_left_wheels_and_support} -0.13" rpy="0 0 0"/>
+			<geometry>
+				<mesh filename="package://wheelchair/meshes/middle_wheel_left.dae"/>
+			</geometry>
 		</visual>
 	</link>
@@ -145,5 +172,5 @@
 		<inertial>
 		<mass value="${rear_wheel_support_mass}"/>
-		<origin xyz="0 0 0" rpy="0 1.5707 1.5707"/>
+		<origin xyz="0 0 0" rpy="0 0 0"/>
 		<inertia
 			ixx="0.1" ixy="0.0" ixz="0.0"
@@ -169,5 +196,5 @@
 		<inertial>
 		<mass value="${rear_wheel_support_mass}"/>
-		<origin xyz="0 0 0" rpy="0 1.5707 1.5707"/>
+		<origin xyz="0 0 0" rpy="0 0 0"/>
 		<inertia
 			ixx="0.1" ixy="0.0" ixz="0.0"
@@ -197,4 +224,12 @@
 		<child link="chassis" />
 	</joint>
+	<joint type="prismatic" name="upper_chassis_joint">
+		<origin xyz="${x_upper_chassis} ${y_upper_chassis} ${y_upper_chassis}" rpy="0 0 0" />
+		<parent link="chassis"/>
+		<child link="upper_chassis" />
+		<axis xyz="0 0 1"/>
+		<limit effort="10000" velocity="1000" />
+		<dynamics damping="1.0" friction="1.0" />
+  	</joint>
 	<joint type="continuous" name="left_wheel_front_joint">
 		<origin xyz="0.523 ${y_left_wheels_and_support} 0.13" rpy="0 0 0" />
@@ -245,4 +280,15 @@
 		<dynamics damping="1.0" friction="1.0" />
   	</joint>
+	<!-- ******** Define Transmissions ********** -->
+	<transmission name="upper_chassis_trans">
+		<type>transmission_interface/SimpleTransmission</type>
+		<actuator name="upper_chassis_motor">
+			<hardwareInterface>EffortJointInterface</hardwareInterface>
+			<mechanicalReduction>1</mechanicalReduction>
+		</actuator>
+		<joint name="upper_chassis_joint">
+			<hardwareInterface>EffortJointInterface</hardwareInterface>
+		</joint>
+ 	</transmission>
 	<transmission name="left_wheel_trans">
 		<type>transmission_interface/SimpleTransmission</type>
@@ -252,5 +298,5 @@
 		</actuator>
 		<joint name="left_wheel_front_joint">
-		<hardwareInterface>VelocityJointInterface</hardwareInterface>
+			<hardwareInterface>VelocityJointInterface</hardwareInterface>
 		</joint>
  	</transmission>
@@ -262,5 +308,5 @@
 		</actuator>
 		<joint name="right_wheel_front_joint">
-		<hardwareInterface>VelocityJointInterface</hardwareInterface>
+			<hardwareInterface>VelocityJointInterface</hardwareInterface>
 		</joint>
  	</transmission>

Commit message: prismatic not working

File: urdf/wheelchair.xacro (robot description, xacro)
@@ -60,5 +60,5 @@
 		</inertial>
 		<collision>
-			<origin xyz="-${x_upper_chassis} -${y_upper_chassis} -${y_upper_chassis}" rpy="0 0 0"/>
+			<origin xyz="-${x_upper_chassis} -${y_upper_chassis} -${z_upper_chassis}" rpy="0 0 0"/>
 			<geometry>
 				<mesh filename="package://wheelchair/meshes/upper_chassis.dae"/>
@@ -66,5 +66,5 @@
 		</collision>
 		<visual>
-			<origin xyz="-${x_upper_chassis} -${y_upper_chassis} -${y_upper_chassis}" rpy="0 0 0"/>
+			<origin xyz="-${x_upper_chassis} -${y_upper_chassis} -${z_upper_chassis}" rpy="0 0 0"/>
 			<geometry>
 				<mesh filename="package://wheelchair/meshes/upper_chassis.dae"/>
@@ -225,10 +225,9 @@
 	</joint>
 	<joint type="prismatic" name="upper_chassis_joint">
-		<origin xyz="${x_upper_chassis} ${y_upper_chassis} ${y_upper_chassis}" rpy="0 0 0" />
+		<origin xyz="${x_upper_chassis} ${y_upper_chassis} ${z_upper_chassis}" rpy="0 0 0" />
 		<parent link="chassis"/>
 		<child link="upper_chassis" />
 		<axis xyz="0 0 1"/>
-		<limit effort="10000" velocity="1000" />
-		<dynamics damping="1.0" friction="1.0" />
+		<limit effort="10000" lower="0.0" upper="1.0" velocity="1.0"/>
   	</joint>
 	<joint type="continuous" name="left_wheel_front_joint">
@@ -277,5 +276,5 @@
 		<child link="right_wheel_back" />
 		<axis xyz="0 1 0" rpy="0 0 0" />
-		<limit effort="10000" velocity="1000" />
+		<limit effort="10000" velocity="1000"/>
 		<dynamics damping="1.0" friction="1.0" />
   	</joint>

Commit message: prismatic joint of upper chassis link working

File: urdf/wheelchair.xacro (robot description, xacro)
@@ -229,5 +229,5 @@
 		<child link="upper_chassis" />
 		<axis xyz="0 0 1"/>
-		<limit effort="10000" lower="0.0" upper="1.0" velocity="1.0"/>
+		<limit effort="10000" lower="0.0" upper="0.045" velocity="0.01"/>
   	</joint>
 	<joint type="continuous" name="left_wheel_front_joint">

Commit message: minor fixes

File: urdf/wheelchair.xacro (robot description, xacro)
@@ -5,6 +5,6 @@
 	<xacro:property name="robot_name" value="wheelchair" />
 	<xacro:property name="chassis_mass" value="50"/>
-	<xacro:property name="upper_chassis_mass" value="30"/>
-	<xacro:property name="middle_wheel_mass" value="15"/>
+	<xacro:property name="upper_chassis_mass" value="20"/>
+	<xacro:property name="middle_wheel_mass" value="10"/>
 	<xacro:property name="middle_wheel_radius" value="0.128"/>
 	<xacro:property name="rear_wheel_radius" value="0.060"/>
@@ -99,23 +99,23 @@
 	<link name="right_wheel">
 		<inertial>
-		<mass value="${middle_wheel_mass}"/>
-		<origin xyz="0 0 0" rpy="0 1.5707 1.5707"/>
-		<inertia
+			<mass value="${middle_wheel_mass}"/>
+			<origin xyz="0 0 0" rpy="0 1.5707 1.5707"/>
+			<inertia
 			ixx="0.1" ixy="0.0" ixz="0.0"
 			iyy="0.1" iyz="0.0"
 			izz="0.1"
-		/>
-		</inertial>
-		<collision>
-		<origin xyz="0 0 0" rpy="0 1.5707 1.5707"/>
-		<geometry>
-			<cylinder radius="${middle_wheel_radius}" length="0.05"/>
-		</geometry>
-		</collision>
-		<visual>
-		<origin xyz="-0.523 -${y_right_wheels_and_support} -0.13" rpy="0 0 0"/>
-		<geometry>
-			<mesh filename="package://wheelchair/meshes/middle_wheel_right.dae"/>
-		</geometry>
+			/>
+		</inertial>
+		<collision>
+			<origin xyz="0 0 0" rpy="0 1.5707 1.5707"/>
+			<geometry>
+				<cylinder radius="${middle_wheel_radius}" length="0.05"/>
+			</geometry>
+		</collision>
+		<visual>
+			<origin xyz="-0.523 -${y_right_wheels_and_support} -0.13" rpy="0 0 0"/>
+			<geometry>
+				<mesh filename="package://wheelchair/meshes/middle_wheel_right.dae"/>
+			</geometry>
 		</visual>
 	</link>
@@ -123,23 +123,23 @@
 	<link name="right_wheel_back">
 		<inertial>
-		<mass value="${rear_wheel_mass}"/>
-		<origin xyz="0 0 0" rpy="0 1.5707 1.5707"/>
-		<inertia
-			ixx="0.1" ixy="0.0" ixz="0.0"
-			iyy="0.1" iyz="0.0"
-			izz="0.1"
-		/>
-		</inertial>
-		<collision>
-		<origin xyz="0 0 0" rpy="0 1.5707 1.5707"/>
-		<geometry>
-			<cylinder radius="${rear_wheel_radius}" length="${rear_wheel_length}"/>
-		</geometry>
-		</collision>
-		<visual>
-		<origin xyz="-${x_back_wheel} -${y_right_wheels_and_support} -${z_back_wheel}" rpy="0 0 0"/>
-		<geometry>
-			<mesh filename="package://wheelchair/meshes/right_wheel_back.dae"/>
-		</geometry>
+			<mass value="${rear_wheel_mass}"/>
+			<origin xyz="0 0 0" rpy="0 1.5707 1.5707"/>
+			<inertia
+				ixx="0.1" ixy="0.0" ixz="0.0"
+				iyy="0.1" iyz="0.0"
+				izz="0.1"
+			/>
+		</inertial>
+		<collision>
+			<origin xyz="0 0 0" rpy="0 1.5707 1.5707"/>
+			<geometry>
+				<cylinder radius="${rear_wheel_radius}" length="${rear_wheel_length}"/>
+			</geometry>
+		</collision>
+		<visual>
+			<origin xyz="-${x_back_wheel} -${y_right_wheels_and_support} -${z_back_wheel}" rpy="0 0 0"/>
+			<geometry>
+				<mesh filename="package://wheelchair/meshes/right_wheel_back.dae"/>
+			</geometry>
 		</visual>
 	</link>
@@ -147,23 +147,23 @@
 	<link name="left_wheel_back">
 		<inertial>
-		<mass value="${rear_wheel_mass}"/>
-		<origin xyz="0 0 0" rpy="0 1.5707 1.5707"/>
-		<inertia
-			ixx="0.1" ixy="0.0" ixz="0.0"
-			iyy="0.1" iyz="0.0"
-			izz="0.1"
-		/>
-		</inertial>
-		<collision>
-		<origin xyz="0 0 0" rpy="0 1.5707 1.5707"/>
-		<geometry>
-			<cylinder radius="${rear_wheel_radius}" length="${rear_wheel_length}"/>
-		</geometry>
-		</collision>
-		<visual>
-		<origin xyz="-${x_back_wheel} -${y_left_wheels_and_support} -${z_back_wheel}" rpy="0 0 0"/>
-		<geometry>
-			<mesh filename="package://wheelchair/meshes/left_wheel_back.dae"/>
-		</geometry>
+			<mass value="${rear_wheel_mass}"/>
+			<origin xyz="0 0 0" rpy="0 1.5707 1.5707"/>
+			<inertia
+				ixx="0.1" ixy="0.0" ixz="0.0"
+				iyy="0.1" iyz="0.0"
+				izz="0.1"
+			/>
+		</inertial>
+		<collision>
+			<origin xyz="0 0 0" rpy="0 1.5707 1.5707"/>
+			<geometry>
+				<cylinder radius="${rear_wheel_radius}" length="${rear_wheel_length}"/>
+			</geometry>
+		</collision>
+		<visual>
+			<origin xyz="-${x_back_wheel} -${y_left_wheels_and_support} -${z_back_wheel}" rpy="0 0 0"/>
+			<geometry>
+				<mesh filename="package://wheelchair/meshes/left_wheel_back.dae"/>
+			</geometry>
 		</visual>
 	</link>
@@ -171,23 +171,23 @@
 	<link name="left_wheel_support">
 		<inertial>
-		<mass value="${rear_wheel_support_mass}"/>
-		<origin xyz="0 0 0" rpy="0 0 0"/>
-		<inertia
-			ixx="0.1" ixy="0.0" ixz="0.0"
-			iyy="0.1" iyz="0.0"
-			izz="0.1"
-		/>
-		</inertial>
-		<collision>
-		<origin xyz="-${x_wheel_support} -${y_left_wheels_and_support} -${z_wheel_support}" rpy="0 0 0"/>
-		<geometry>
-			<mesh filename="package://wheelchair/meshes/left_wheel_support.dae"/>
-		</geometry>
-		</collision>
-		<visual>
-		<origin xyz="-${x_wheel_support} -${y_left_wheels_and_support} -${z_wheel_support}" rpy="0 0 0"/>
-		<geometry>
-			<mesh filename="package://wheelchair/meshes/left_wheel_support.dae"/>
-		</geometry>
+			<mass value="${rear_wheel_support_mass}"/>
+			<origin xyz="0 0 0" rpy="0 0 0"/>
+			<inertia
+				ixx="0.1" ixy="0.0" ixz="0.0"
+				iyy="0.1" iyz="0.0"
+				izz="0.1"
+			/>
+		</inertial>
+		<collision>
+			<origin xyz="-${x_wheel_support} -${y_left_wheels_and_support} -${z_wheel_support}" rpy="0 0 0"/>
+			<geometry>
+				<mesh filename="package://wheelchair/meshes/left_wheel_support.dae"/>
+			</geometry>
+		</collision>
+		<visual>
+			<origin xyz="-${x_wheel_support} -${y_left_wheels_and_support} -${z_wheel_support}" rpy="0 0 0"/>
+			<geometry>
+				<mesh filename="package://wheelchair/meshes/left_wheel_support.dae"/>
+			</geometry>
 		</visual>
 	</link>
@@ -195,23 +195,23 @@
 	<link name="right_wheel_support">
 		<inertial>
-		<mass value="${rear_wheel_support_mass}"/>
-		<origin xyz="0 0 0" rpy="0 0 0"/>
-		<inertia
-			ixx="0.1" ixy="0.0" ixz="0.0"
-			iyy="0.1" iyz="0.0"
-			izz="0.1"
-		/>
-		</inertial>
-		<collision>
-		<origin xyz="-${x_wheel_support} -${y_right_wheels_and_support} -${z_wheel_support}" rpy="0 0 0"/>
-		<geometry>
-			<mesh filename="package://wheelchair/meshes/right_wheel_support.dae"/>
-		</geometry>
-		</collision>
-		<visual>
-		<origin xyz="-${x_wheel_support} -${y_right_wheels_and_support} -${z_wheel_support}" rpy="0 0 0"/>
-		<geometry>
-			<mesh filename="package://wheelchair/meshes/right_wheel_support.dae"/>
-		</geometry>
+			<mass value="${rear_wheel_support_mass}"/>
+			<origin xyz="0 0 0" rpy="0 0 0"/>
+			<inertia
+				ixx="0.1" ixy="0.0" ixz="0.0"
+				iyy="0.1" iyz="0.0"
+				izz="0.1"
+			/>
+		</inertial>
+		<collision>
+			<origin xyz="-${x_wheel_support} -${y_right_wheels_and_support} -${z_wheel_support}" rpy="0 0 0"/>
+			<geometry>
+				<mesh filename="package://wheelchair/meshes/right_wheel_support.dae"/>
+			</geometry>
+		</collision>
+		<visual>
+			<origin xyz="-${x_wheel_support} -${y_right_wheels_and_support} -${z_wheel_support}" rpy="0 0 0"/>
+			<geometry>
+				<mesh filename="package://wheelchair/meshes/right_wheel_support.dae"/>
+			</geometry>
 		</visual>
 	</link>
@@ -225,5 +225,5 @@
 	</joint>
 	<joint type="prismatic" name="upper_chassis_joint">
-		<origin xyz="${x_upper_chassis} ${y_upper_chassis} ${z_upper_chassis}" rpy="0 0 0" />
+		<origin xyz="${x_upper_chassis} ${y_upper_chassis} 0.37" rpy="0 0 0" />
 		<parent link="chassis"/>
 		<child link="upper_chassis" />

Commit message: added back mesh and revolute joint

File: urdf/wheelchair.xacro (robot description, xacro)
@@ -5,5 +5,6 @@
 	<xacro:property name="robot_name" value="wheelchair" />
 	<xacro:property name="chassis_mass" value="50"/>
-	<xacro:property name="upper_chassis_mass" value="20"/>
+	<xacro:property name="upper_chassis_mass" value="15"/>
+	<xacro:property name="back_mass" value="5"/>
 	<xacro:property name="middle_wheel_mass" value="10"/>
 	<xacro:property name="middle_wheel_radius" value="0.128"/>
@@ -24,4 +25,10 @@
 	<xacro:property name="y_upper_chassis" value="0.29"/>
 	<xacro:property name="z_upper_chassis" value="0.4"/>
+	<xacro:property name="x_back" value="0.17"/>
+	<xacro:property name="y_back" value="0.29"/>
+	<xacro:property name="z_back" value="0.45"/>
+	<xacro:property name="x_back_joint" value="0.25"/>
+	<xacro:property name="y_back_joint" value="0.0"/>
+	<xacro:property name="z_back_joint" value="0.051"/>
 	<!-- Make Chassis of Bot -->
 	<link name="chassis">
@@ -62,5 +69,5 @@
 			<origin xyz="-${x_upper_chassis} -${y_upper_chassis} -${z_upper_chassis}" rpy="0 0 0"/>
 			<geometry>
-				<mesh filename="package://wheelchair/meshes/upper_chassis.dae"/>
+				<mesh filename="package://wheelchair/meshes/upper_chassis_no_back.dae"/>
 			</geometry>
 		</collision>
@@ -68,5 +75,28 @@
 			<origin xyz="-${x_upper_chassis} -${y_upper_chassis} -${z_upper_chassis}" rpy="0 0 0"/>
 			<geometry>
-				<mesh filename="package://wheelchair/meshes/upper_chassis.dae"/>
+				<mesh filename="package://wheelchair/meshes/upper_chassis_no_back.dae"/>
+			</geometry>
+		</visual>
+	</link>
+	<link name="back">
+		<inertial>
+			<mass value="${back_mass}"/>
+      		<origin xyz="0 0 0" rpy=" 0 0 0"/>
+      		<inertia
+      			ixx="0.147116667" ixy="0" ixz="0"
+      			iyy="0.334951167" iyz="0"
+      			izz="0.3978345"
+      		/>
+		</inertial>
+		<collision>
+			<origin xyz="-${x_back} -${y_back} -${z_back}" rpy="0 0 0"/>
+			<geometry>
+				<mesh filename="package://wheelchair/meshes/back.dae"/>
+			</geometry>
+		</collision>
+		<visual>
+			<origin xyz="-${x_back} -${y_back} -${z_back}" rpy="0 0 0"/>
+			<geometry>
+				<mesh filename="package://wheelchair/meshes/back.dae"/>
 			</geometry>
 		</visual>
@@ -225,9 +255,18 @@
 	</joint>
 	<joint type="prismatic" name="upper_chassis_joint">
-		<origin xyz="${x_upper_chassis} ${y_upper_chassis} 0.37" rpy="0 0 0" />
+		<!--<origin xyz="${x_upper_chassis} ${y_upper_chassis} ${z_upper_chassis}" rpy="0 0 0" />-->
+		<origin xyz="${x_upper_chassis} ${y_upper_chassis} 0.38" rpy="0 0 0" />-
 		<parent link="chassis"/>
 		<child link="upper_chassis" />
 		<axis xyz="0 0 1"/>
 		<limit effort="10000" lower="0.0" upper="0.045" velocity="0.01"/>
+  	</joint>
+	<joint type="revolute" name="back_joint">
+		<origin xyz="-${x_back_joint} ${y_back_joint} ${z_back_joint}" rpy="0 0 0"/>
+		<parent link="upper_chassis"/>
+		<child link="back" />
+		<axis xyz="0 1 0"/>
+		<limit effort="10000" velocity="10" upper="0" lower="0"/>
+		<dynamics damping="1.0" friction="1.0" />
   	</joint>
 	<joint type="continuous" name="left_wheel_front_joint">
@@ -290,4 +329,14 @@
 		</joint>
  	</transmission>
+	<transmission name="back_trans">
+		<type>transmission_interface/SimpleTransmission</type>
+		<actuator name="back_motor">
+			<hardwareInterface>EffortJointInterface</hardwareInterface>
+			<mechanicalReduction>1</mechanicalReduction>
+		</actuator>
+		<joint name="back_joint">
+			<hardwareInterface>EffortJointInterface</hardwareInterface>
+		</joint>
+	</transmission>
 	<transmission name="left_wheel_trans">
 		<type>transmission_interface/SimpleTransmission</type>

Commit message: revolut back joint working

File: urdf/wheelchair.xacro (robot description, xacro)
@@ -4,8 +4,8 @@
 	<!--<xacro:include filename="$(find wheelchair)/urdf/wheelchair.gazebo" />-->
 	<xacro:property name="robot_name" value="wheelchair" />
-	<xacro:property name="chassis_mass" value="50"/>
-	<xacro:property name="upper_chassis_mass" value="15"/>
+	<xacro:property name="chassis_mass" value="60"/>
+	<xacro:property name="upper_chassis_mass" value="20"/>
 	<xacro:property name="back_mass" value="5"/>
-	<xacro:property name="middle_wheel_mass" value="10"/>
+	<xacro:property name="middle_wheel_mass" value="15"/>
 	<xacro:property name="middle_wheel_radius" value="0.128"/>
 	<xacro:property name="rear_wheel_radius" value="0.060"/>
@@ -260,5 +260,5 @@
 		<child link="upper_chassis" />
 		<axis xyz="0 0 1"/>
-		<limit effort="10000" lower="0.0" upper="0.045" velocity="0.01"/>
+		<limit effort="10000" lower="0.0" upper="0.045" velocity="1.0"/>
   	</joint>
 	<joint type="revolute" name="back_joint">
@@ -267,5 +267,5 @@
 		<child link="back" />
 		<axis xyz="0 1 0"/>
-		<limit effort="10000" velocity="10" upper="0" lower="0"/>
+		<limit effort="10000" velocity="1.0" upper="0.3" lower="-1.0"/>
 		<dynamics damping="1.0" friction="1.0" />
   	</joint>

Commit message: devel of up_down_motor_sync

File: urdf/wheelchair.xacro (robot description, xacro)
@@ -4,5 +4,5 @@
 	<!--<xacro:include filename="$(find wheelchair)/urdf/wheelchair.gazebo" />-->
 	<xacro:property name="robot_name" value="wheelchair" />
-	<xacro:property name="chassis_mass" value="60"/>
+	<xacro:property name="chassis_mass" value="100"/>
 	<xacro:property name="upper_chassis_mass" value="20"/>
 	<xacro:property name="back_mass" value="5"/>

Commit message: up_down_sync

File: urdf/wheelchair.xacro (robot description, xacro)
@@ -15,5 +15,5 @@
 	<!-- Axis Values-->
 	<xacro:property name="z_wheel_support" value="0.125"/>
-	<xacro:property name="z_back_wheel" value="0.062"/>
+	<xacro:property name="z_back_wheel" value="0.063"/>
 	<xacro:property name="z_back_diff" value="-0.063"/> <!-- Equals to: (z_back_wheel - z_wheel_support) -->
 	<xacro:property name="x_wheel_support" value="0.083"/>

Commit message: upd

File: urdf/wheelchair.xacro (robot description, xacro)
@@ -8,12 +8,13 @@
 	<xacro:property name="back_mass" value="5"/>
 	<xacro:property name="middle_wheel_mass" value="15"/>
-	<xacro:property name="middle_wheel_radius" value="0.128"/>
+	<xacro:property name="middle_wheel_radius" value="0.13"/>
+	<xacro:property name="middle_wheel_length" value="0.07"/>
 	<xacro:property name="rear_wheel_radius" value="0.060"/>
 	<xacro:property name="rear_wheel_length" value="0.025"/>
-	<xacro:property name="rear_wheel_mass" value="3"/>
+	<xacro:property name="rear_wheel_mass" value="4"/>
 	<xacro:property name="rear_wheel_support_mass" value="2"/>
 	<!-- Axis Values-->
 	<xacro:property name="z_wheel_support" value="0.125"/>
-	<xacro:property name="z_back_wheel" value="0.063"/>
+	<xacro:property name="z_back_wheel" value="0.06"/>
 	<xacro:property name="z_back_diff" value="-0.063"/> <!-- Equals to: (z_back_wheel - z_wheel_support) -->
 	<xacro:property name="x_wheel_support" value="0.083"/>
@@ -22,4 +23,5 @@
 	<xacro:property name="y_right_wheels_and_support" value="0.051"/>
 	<xacro:property name="y_left_wheels_and_support" value="0.527"/>
+	<xacro:property name="z_mid_wheels" value="0.13"/>
 	<xacro:property name="x_upper_chassis" value="0.42"/>
 	<xacro:property name="y_upper_chassis" value="0.29"/>
@@ -114,11 +116,11 @@
 		</inertial>
 		<collision>
-			<origin xyz="0 0 0" rpy="0 1.5707 1.5707"/>
-			<geometry>
-				<cylinder radius="${middle_wheel_radius}" length="0.05"/>
-			</geometry>
-		</collision>
-		<visual>
-			<origin xyz="-0.523 -${y_left_wheels_and_support} -0.13" rpy="0 0 0"/>
+			<origin xyz="0 0 -0.001" rpy="0 1.5707 1.5707"/>
+			<geometry>
+				<cylinder radius="${middle_wheel_radius}" length="${middle_wheel_length}"/>
+			</geometry>
+		</collision>
+		<visual>
+			<origin xyz="-0.523 -${y_left_wheels_and_support} -${z_mid_wheels}" rpy="0 0 0"/>
 			<geometry>
 				<mesh filename="package://wheelchair/meshes/middle_wheel_left.dae"/>
@@ -138,11 +140,11 @@
 		</inertial>
 		<collision>
-			<origin xyz="0 0 0" rpy="0 1.5707 1.5707"/>
-			<geometry>
-				<cylinder radius="${middle_wheel_radius}" length="0.05"/>
-			</geometry>
-		</collision>
-		<visual>
-			<origin xyz="-0.523 -${y_right_wheels_and_support} -0.13" rpy="0 0 0"/>
+			<origin xyz="0 0 -0.001" rpy="0 1.5707 1.5707"/>
+			<geometry>
+				<cylinder radius="${middle_wheel_radius}" length="${middle_wheel_length}"/>
+			</geometry>
+		</collision>
+		<visual>
+			<origin xyz="-0.523 -${y_right_wheels_and_support} -${z_mid_wheels}" rpy="0 0 0"/>
 			<geometry>
 				<mesh filename="package://wheelchair/meshes/middle_wheel_right.dae"/>
