Commit message: devel dt up_down_motor

File: urdf/wheelchair.xacro (robot description, xacro)
@@ -4,17 +4,17 @@
 	<!--<xacro:include filename="$(find wheelchair)/urdf/wheelchair.gazebo" />-->
 	<xacro:property name="robot_name" value="wheelchair" />
-	<xacro:property name="chassis_mass" value="100"/>
+	<xacro:property name="chassis_mass" value="60"/>
 	<xacro:property name="upper_chassis_mass" value="20"/>
 	<xacro:property name="back_mass" value="5"/>
 	<xacro:property name="middle_wheel_mass" value="15"/>
-	<xacro:property name="middle_wheel_radius" value="0.13"/>
-	<xacro:property name="middle_wheel_length" value="0.07"/>
+	<xacro:property name="middle_wheel_radius" value="0.128"/>
+	<xacro:property name="middle_wheel_length" value="0.05"/>
 	<xacro:property name="rear_wheel_radius" value="0.060"/>
 	<xacro:property name="rear_wheel_length" value="0.025"/>
-	<xacro:property name="rear_wheel_mass" value="4"/>
+	<xacro:property name="rear_wheel_mass" value="3"/>
 	<xacro:property name="rear_wheel_support_mass" value="2"/>
 	<!-- Axis Values-->
 	<xacro:property name="z_wheel_support" value="0.125"/>
-	<xacro:property name="z_back_wheel" value="0.06"/>
+	<xacro:property name="z_back_wheel" value="0.062"/>
 	<xacro:property name="z_back_diff" value="-0.063"/> <!-- Equals to: (z_back_wheel - z_wheel_support) -->
 	<xacro:property name="x_wheel_support" value="0.083"/>
@@ -116,5 +116,5 @@
 		</inertial>
 		<collision>
-			<origin xyz="0 0 -0.001" rpy="0 1.5707 1.5707"/>
+			<origin xyz="0 0 0" rpy="0 1.5707 1.5707"/>
 			<geometry>
 				<cylinder radius="${middle_wheel_radius}" length="${middle_wheel_length}"/>
@@ -140,5 +140,5 @@
 		</inertial>
 		<collision>
-			<origin xyz="0 0 -0.001" rpy="0 1.5707 1.5707"/>
+			<origin xyz="0 0 0" rpy="0 1.5707 1.5707"/>
 			<geometry>
 				<cylinder radius="${middle_wheel_radius}" length="${middle_wheel_length}"/>

Commit message: v1 com pos

File: urdf/wheelchair.xacro (robot description, xacro)
@@ -263,4 +263,5 @@
 		<axis xyz="0 0 1"/>
 		<limit effort="10000" lower="0.0" upper="0.045" velocity="1.0"/>
+		<dynamics damping="1.0" friction="1.0" />
   	</joint>
 	<joint type="revolute" name="back_joint">
@@ -269,5 +270,5 @@
 		<child link="back" />
 		<axis xyz="0 1 0"/>
-		<limit effort="10000" velocity="1.0" upper="0.3" lower="-1.0"/>
+		<limit effort="10000" velocity="1.0" upper="1.0" lower="-0.5773"/>
 		<dynamics damping="1.0" friction="1.0" />
   	</joint>

Commit message: back and up_down sync working 90%

File: urdf/wheelchair.xacro (robot description, xacro)
@@ -270,5 +270,5 @@
 		<child link="back" />
 		<axis xyz="0 1 0"/>
-		<limit effort="10000" velocity="1.0" upper="1.0" lower="-0.5773"/>
+		<limit effort="10000" velocity="1.0" upper="0.8" lower="-0.5773"/>
 		<dynamics damping="1.0" friction="1.0" />
   	</joint>
