Commit message: updates

File: urdf/wheelchair.urdf (robot description, URDF)
Before this commit: robot wheelchair, 10 links, 9 joints
Links:
- link back: mass 5 -> 5.0
- link chassis: mass 60 -> 60.0
- link left_wheel: mass 15 -> 15.0
- link left_wheel_back: mass 3 -> 3.0
- link left_wheel_support: mass 2 -> 2.0
- link right_wheel: mass 15 -> 15.0
- link right_wheel_back: mass 3 -> 3.0
- link right_wheel_support: mass 2 -> 2.0
- link upper_chassis: mass 20 -> 20.0

File: urdf/wheelchair.xacro (robot description, xacro)
@@ -4,14 +4,14 @@
 	<!-- Measurement Values -->
 	<xacro:property name="robot_name" value="wheelchair" />
-	<xacro:property name="chassis_mass" value="60"/>
-	<xacro:property name="upper_chassis_mass" value="20"/>
-	<xacro:property name="back_mass" value="5"/>
-	<xacro:property name="middle_wheel_mass" value="15"/>
+	<xacro:property name="chassis_mass" value="60.0"/>
+	<xacro:property name="upper_chassis_mass" value="20.0"/>
+	<xacro:property name="back_mass" value="5.0"/>
+	<xacro:property name="middle_wheel_mass" value="15.0"/>
 	<xacro:property name="middle_wheel_radius" value="0.128"/>
 	<xacro:property name="middle_wheel_length" value="0.05"/>
 	<xacro:property name="rear_wheel_radius" value="0.060"/>
 	<xacro:property name="rear_wheel_length" value="0.025"/>
-	<xacro:property name="rear_wheel_mass" value="3"/>
-	<xacro:property name="rear_wheel_support_mass" value="2"/>
+	<xacro:property name="rear_wheel_mass" value="3.0"/>
+	<xacro:property name="rear_wheel_support_mass" value="2.0"/>
 	<!-- Axis Values-->
 	<xacro:property name="z_wheel_support" value="0.125"/>
